File: The-Unt1tled-TKL.kicad_pcb (KiCad board)
At the start: 2 copper layers, 211 parts, among them J1 USB_C_Receptacle, J2 AVR-ISP-6, SW1 SW_Reset, SW2 SW_Boot, U1 ATmega324A-P, Y1 20MHz

Commit message: Many things
- Figured out grid placement
- Working on part placements
- Changed footprint from MX-Alp Hybrid to MX-Only.
Parts:
- MX1, MX10, MX100, MX11, MX12, MX13, MX14, MX15, MX16, MX17, MX18, MX19, MX2, MX20, MX21, MX22, MX23, MX24, MX25, MX26, MX27, MX28, MX29, MX3, MX31, MX32, MX33, MX35, MX36, MX37, MX38, MX39, MX4, MX40, MX41, MX42, MX43, MX44, MX45, MX46, MX48, MX49, MX5, MX50, MX53, MX54, MX55, MX56, MX57, MX58, MX59, MX6, MX60, MX61, MX62, MX63, MX64, MX67, MX7, MX70, MX71, MX72, MX73, MX74, MX75, MX76, MX77, MX78, MX79, MX8, MX82, MX83, MX9, MX92, MX93, MX94, MX96: footprint MX_Alps_Hybrid:MX-1U-NoLED -> MX_Only:MXOnly-1U-NoLED
- MX101, MX34, MX47, MX95, MX97, MX99: footprint MX_Alps_Hybrid:MX-1.5U-NoLED -> MX_Only:MXOnly-1.5U-NoLED
- MX30: footprint MX_Alps_Hybrid:MX-2U-NoLED -> MX_Only:MXOnly-1U-NoLED
- MX51, MX68, MX84, MX85, MX86, MX88, MX89, MX90, MX91: footprint MX_Alps_Hybrid:MX-1.25U-NoLED -> MX_Only:MXOnly-1.25U-NoLED
- MX52, MX80: footprint MX_Alps_Hybrid:MX-1.75U-NoLED -> MX_Only:MXOnly-1.75U-NoLED
- MX65: footprint MX_Alps_Hybrid:MX-ISO -> MX_Only:MXOnly-ISO-NoLED
- MX66, MX69: footprint MX_Alps_Hybrid:MX-2.25U-NoLED -> MX_Only:MXOnly-2.25U-NoLED
- MX81: footprint MX_Alps_Hybrid:MX-2.75U-NoLED -> MX_Only:MXOnly-2.75U-NoLED
- MX87: footprint MX_Alps_Hybrid:MX-6.25U-NoLED -> MX_Only:MXOnly-6.25U-NoLED
- MX98: footprint MX_Alps_Hybrid:MX-7U-NoLED -> MX_Only:MXOnly-7U-NoLED
- moved J1 1324.7 mm to (651.7, -139.1), turned to 180 degrees
- moved F1 1316.5 mm to (662.2, -135.1)
- moved C2 1306.7 mm to (639.8, -89.5), turned to -90 degrees
- moved D91 1301.9 mm to (639.0, -139.1)
- moved C1 1295.7 mm to (629.4, -89.5), turned to -90 degrees
- moved Y1 1284.3 mm to (634.3, -82.1), turned to -90 degrees
- moved D2 1280.9 mm to (642.1, -113.8), turned to 90 degrees
- moved D1 1274.6 mm to (636.6, -113.8), turned to 90 degrees
- moved R1 1260.4 mm to (668.3, -100.3), turned to 90 degrees
- moved R2 1258.2 mm to (662.8, -107.2), turned to -90 degrees
- moved C3 1257.7 mm to (669.1, -124.8)
- moved C4 1252.5 mm to (661.6, -124.8)
- moved C5 1251.8 mm to (661.6, -116.0)
- moved R3 1246.7 mm to (648.5, -110.3), turned to -90 degrees
- moved R7 1246.4 mm to (635.3, -132.7)
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
Commit message: Part placement and wireing
Placed diodes. Still need to place other parts in their final position. Started wiring.
Parts:
- MX30: footprint MX_Only:MXOnly-1U-NoLED -> MX_Only:MXOnly-2U-NoLED
- moved D80 362.2 mm to (102.4, 96.5)
- moved D81 353.5 mm to (116.7, 96.5)
- moved D82 344.8 mm to (131.0, 96.5)
- moved D83 307.8 mm to (173.8, 96.5)
- moved D67 294.7 mm to (97.6, 92.6)
- moved D68 286.0 mm to (111.9, 92.6)
- moved D69 277.4 mm to (126.2, 92.6)
- moved D70 268.7 mm to (140.5, 92.6)
- moved D71 260.1 mm to (154.8, 92.6)
- moved U1 252.8 mm to (403.2, 75.6)
- moved D72 251.4 mm to (169.1, 92.6)
- moved C2 251.1 mm to (465.9, 91.6)
- moved C5 251.1 mm to (487.7, 65.1)
- moved D91 251.1 mm to (465.2, 42.1)
- moved J1 251.1 mm to (477.8, 42.1)
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Connections:
- C1 pad 2: Net-(U1-XTAL1) -> Net-(U1-PA2)
- C2 pad 2: Net-(U1-XTAL2) -> Net-(U1-PA4)
- D10 pad 1: COL0 -> ROW0
- D11 pad 1: COL0 -> ROW0
- D12 pad 1: COL0 -> ROW0
- D13 pad 1: COL0 -> ROW0
- D14 pad 1: COL0 -> ROW0
- D15 pad 1: COL0 -> ROW0
- D16 pad 1: COL0 -> ROW0
- D17 pad 1: COL0 -> ROW0
- D18 pad 1: COL0 -> ROW0
- D19 pad 1: COL0 -> ROW1
- D20 pad 1: COL0 -> ROW1
- D21 pad 1: COL0 -> ROW1
- D22 pad 1: COL0 -> ROW1
- D23 pad 1: COL0 -> ROW1
- D24 pad 1: COL0 -> ROW1
- D25 pad 1: COL0 -> ROW1
- D26 pad 1: COL0 -> ROW1
- D27 pad 1: COL0 -> ROW1
- D28 pad 1: COL0 -> ROW1
- D29 pad 1: COL0 -> ROW1
- D3 pad 1: COL0 -> ROW0
- D30 pad 1: COL0 -> ROW1
- D31 pad 1: COL0 -> ROW1
- D32 pad 1: COL0 -> ROW1
- D33 pad 1: COL0 -> ROW1
- D34 pad 1: COL0 -> ROW1
- D35 pad 1: COL0 -> ROW1
- D36 pad 1: COL0 -> ROW2
- D37 pad 1: COL0 -> ROW2
- D38 pad 1: COL0 -> ROW2
- D39 pad 1: COL0 -> ROW2
- D4 pad 1: COL0 -> ROW0
- D40 pad 1: COL0 -> ROW2
- D41 pad 1: COL0 -> ROW2
- D42 pad 1: COL0 -> ROW2
- D43 pad 1: COL0 -> ROW2
- D44 pad 1: COL0 -> ROW2
- D45 pad 1: COL0 -> ROW2
- D46 pad 1: COL0 -> ROW2
- D47 pad 1: COL0 -> ROW2
- D48 pad 1: COL0 -> ROW2
- D49 pad 1: COL0 -> ROW2
- D5 pad 1: COL0 -> ROW0
- D50 pad 1: COL0 -> ROW2
- D51 pad 1: COL0 -> ROW2
- D52 pad 1: COL0 -> ROW2
- D53 pad 1: COL0 -> ROW3
- D54 pad 1: COL0 -> ROW3
- D55 pad 1: COL0 -> ROW3
- D56 pad 1: COL0 -> ROW3
- D57 pad 1: COL0 -> ROW3
- D58 pad 1: COL0 -> ROW3
- D59 pad 1: COL0 -> ROW3
- D6 pad 1: COL0 -> ROW0
- D60 pad 1: COL0 -> ROW3
- D61 pad 1: COL0 -> ROW3
- D62 pad 1: COL0 -> ROW3
- D63 pad 1: COL0 -> ROW3
- D64 pad 1: COL0 -> ROW3
- D65 pad 1: COL0 -> ROW3
- D66 pad 1: COL0 -> ROW3
- D7 pad 1: COL0 -> ROW0
- D8 pad 1: COL0 -> ROW0
- D9 pad 1: COL0 -> ROW0
- U1 pad 12: Net-(U1-XTAL2) -> unconnected-(U1-XTAL2-Pad12)
- U1 pad 13: Net-(U1-XTAL1) -> unconnected-(U1-XTAL1-Pad13)
- U1 pad 16: D+ -> unconnected-(U1-PD2-Pad16)
- U1 pad 17: D- -> unconnected-(U1-PD3-Pad17)
- U1 pad 20: boot -> unconnected-(U1-PD6-Pad20)
- U1 pad 30: +5V -> unconnected-(U1-AVCC-Pad30)
- U1 pad 36: unconnected-(U1-PA4-Pad36) -> Net-(U1-PA4)
- U1 pad 38: unconnected-(U1-PA2-Pad38) -> Net-(U1-PA2)
- U1 pad 40: unconnected-(U1-PA0-Pad40) -> reset
- U1 pad 6: MOSI -> unconnected-(U1-PB5-Pad6)
- U1 pad 7: MISO -> unconnected-(U1-PB6-Pad7)
- U1 pad 8: SCK -> unconnected-(U1-PB7-Pad8)
- U1 pad 9: reset -> unconnected-(U1-~{RESET}-Pad9)
- Y1 pad 1: Net-(U1-XTAL1) -> Net-(U1-PA2)
- Y1 pad 3: Net-(U1-XTAL2) -> Net-(U1-PA4)
Routing:
- net COL0: track 0.00 -> 133.5 mm
- net COL5: track 0.00 -> 128.6 mm
- net COL2: track 0.00 -> 121.8 mm
- net COL4: track 0.00 -> 96.1 mm
- net COL3: track 0.00 -> 96.1 mm
- net COL1: track 0.00 -> 95.3 mm
- net Net-(D83-A): track 0.00 -> 11.9 mm
Other:
- board outline added: 462.8 x 192.9 mm
